File: Big Muff.kicad_pcb (KiCad board)
At the start: 2 copper layers, 48.3 x 45.7 mm, 46 parts, among them J1 Power, J2 Input, J3 Output, J4 LED, J5 ToneSwitch, U1 TL074

Commit message: Fixed footprint for resistors, re-placed components
Parts:
- R1, R10, R11, R12, R13, R14, R15, R16, R17, R18, R19, R2, R3, R4, R5, R6, R7, R8, R9: footprint Resistor_THT:R_Axial_DIN0204_L3.6mm_D1.6mm_P5.08mm_Horizontal -> Resistor_THT:R_Axial_DIN0204_L3.6mm_D1.6mm_P7.62mm_Horizontal
- moved C7 11.3 mm to (137.2, 66.1)
- moved R3 5.08 mm to (132.1, 63.5)
- moved C1 4.58 mm to (137.2, 72.4)
- moved C5 4.58 mm to (134.7, 59.7)
- moved C4 4.56 mm to (134.7, 54.6)
- moved C2 3.62 mm to (137.2, 78.8)
- moved J5 2.54 mm to (124.5, 94.0)
- moved J4 2.54 mm to (134.6, 94.0)
- moved R1 2.54 mm to (124.5, 58.4)
- moved R14 2.54 mm to (124.5, 76.2)
- moved R2 2.54 mm to (124.5, 61.0)
- moved R4 2.54 mm to (124.5, 66.0)
- moved R5 2.54 mm to (124.5, 68.6)
- moved R6 2.54 mm to (124.5, 81.3)
- moved R7 2.54 mm to (124.5, 71.1)
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Other:
- board text added: "BIG MUFF PI FRANK SINAPI JULY 2026"
- board text added: "INPUT"
- board text added: "OUT"
- board text added: "PWR"
